File: amplifone-sega-adapter.kicad_pcb (KiCad board)
At the start: 2 copper layers, 101.6 x 101.6 mm, 94 parts, among them J0 Conn_01x03_Male, J1 640385-4, J2 640385-4, J3 640385-4, J4 640385-4, U1 TL082, U2 TL082, U3 TL082, U4 TL082, U5 TL082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

Commit message: revision 2
Parts:
- U6, U7, U8: footprint Package_TO_SOT_THT:TO-92_Inline -> Package_TO_SOT_THT:TO-92
Routing:
- net Net-(U1B--): track 24.6 -> 29.2 mm
- net /amplifiers/Y_IN: track 66.2 -> 70.0 mm
- net /amplifiers/R_IN: track 92.0 -> 89.1 mm
- net /amplifiers/X_OUT: track 60.0 -> 62.9 mm
- net -9V: track 204.2 -> 207.0 mm
- net /amplifiers/B_IN: track 58.7 -> 56.4 mm
- net +9V: track 171.6 -> 173.9 mm
- net /amplifiers/G_IN: track 76.2 -> 78.0 mm
- net +0V5: track 117.7 -> 119.4 mm
- net -12V: track 13.5 -> 12.3 mm
