File: amplifone-sega-adapter-amps.kicad_sch (KiCad schematic)
At the start: 93 parts, among them J1 640385-4, J2 640385-4, J3 640385-4, J4 640385-4, U1 TL082, U2 TL082, U3 TL082, U4 TL082, U5 TL082, U6 MCP1702-1502E/TO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

Commit message: Add files via upload
Other:
- moved on the sheet: J1, J2, J3, J4
